File: doc/kicad/CAN-BUS-Weichendecoder/CAN-BUS-Weichendecoder.sch (KiCad schematic (older format))
At the start: 37 parts, among them J1 RJ45_LED_Shielded, J10 Conn_01x06_Female, J11 Conn_01x06_Female, J12 Conn_01x06_Female, J13 Conn_01x06_Female, J2 RJ45_Shielded, J3 Power, J4 Weiche 1, J5 Weiche 2, J6 Weiche 3, J7 Weiche 4, J8 Weiche 5, J9 Power Weiche, K1 HFD2_005-S-L2-D, U1 ULN2803A, U2 ULN2803A, U3 PCF8574, U4 PCF8574, U5 PCF8574, U6 ULN2803A, U7 ULN2803A, U8 ULN2803A

Commit message: Aktueller Stand
Parts:
- added J?: Conn_01x07_Female, symbol Connector:Conn_01x07_Female
Connections:
- wire segments 227 -> 229
Other:
- moved on the sheet: Shield1
Changed lines of the file:
@@
 L CAN-BUS-MODULE-TJA1050:CAN-BUS_MODULE_TJA1050 Shield1
 U 1 1 60585225
-P 1900 2850
-F 0 "Shield1" H 1850 2175 50  0000 C CNN
-F 1 "CAN-BUS_MODULE_TJA1050" H 1850 2084 50  0000 C CNN
-F 2 "kicad-lib:MCP2515_CAN_MODULE_BY0-10" H 1900 2850 50  0001 C CIN
-F 3 "" H 1900 2850 50  0001 C CNN
-	1    1900 2850
+P 1700 2850
+F 0 "Shield1" H 1650 2175 50  0000 C CNN
+F 1 "CAN-BUS_MODULE_TJA1050" H 1650 2084 50  0000 C CNN
+F 2 "kicad-lib:MCP2515_CAN_MODULE_BY0-10" H 1700 2850 50  0001 C CIN
+F 3 "" H 1700 2850 50  0001 C CNN
+	1    1700 2850
 	1    0    0    -1
 $EndComp
@@
 	2400 5650 1850 5650
 Wire Wire Line
-	1100 3050 850  3050
+	1100 3050 900  3050
 Wire Wire Line
 	850  3050 850  3850
@@
 Connection ~ 2050 5100
 Wire Wire Line
-	1100 2950 800  2950
+	1100 2950 900  2950
 Wire Wire Line
 	800  2950 800  3900
@@
 Wire Wire Line
 	3950 4900 4400 4900
+Connection ~ 900  3050
+Wire Wire Line
+	900  3050 850  3050
+Connection ~ 900  2950
+$Comp
+L Connector:Conn_01x07_Female J?
+U 1 1 60962CDF
+P 2400 2950
+F 0 "J?" H 2292 2425 50  0000 C CNN
+F 1 "Conn_01x07_Female" H 2292 2516 50  0000 C CNN
+F 2 "" H 2400 2950 50  0001 C CNN
+F 3 "~" H 2400 2950 50  0001 C CNN
+	1    2400 2950
+	-1   0    0    1
+$EndComp
+Wire Wire Line
+	800  2950 900  2950
 $EndSCHEMATC

Commit message: Platine weiterentwickelt, aktueller Arbeitsstand
Parts:
- gave numbers to parts that had none: 1
Connections:
- wire segments 229 -> 253
Other:
- moved on the sheet: U6
Changed lines of the file:
@@
 	1    0    0    -1
 $EndComp
-Wire Wire Line
-	8100 1450 8350 1450
-Wire Wire Line
-	8350 1350 8100 1350
 $Comp
 L Interface_Expansion:PCF8574 U3
@@
 $EndComp
 $Comp
-L Transistor_Array:ULN2803A U6
-U 1 1 60418EE2
-P 8750 1550
-F 0 "U6" H 8750 2117 50  0000 C CNN
-F 1 "ULN2803A" H 8750 2026 50  0000 C CNN
-F 2 "Package_DIP:DIP-18_W7.62mm" H 8800 900 50  0001 L CNN
-F 3 "http://www.ti.com/lit/ds/symlink/uln2803a.pdf" H 8850 1350 50  0001 C CNN
-	1    8750 1550
-	1    0    0    -1
-$EndComp
-Wire Wire Line
-	8100 1550 8350 1550
-Wire Wire Line
-	8100 1650 8350 1650
-Wire Wire Line
-	8350 1750 8100 1750
-Wire Wire Line
-	8100 1850 8350 1850
-Wire Wire Line
-	8100 1950 8350 1950
-Wire Wire Line
-	8100 2050 8350 2050
-$Comp
 L MCU_Module:Arduino_Nano_v3.x A1
 U 1 1 60416171
@@
 L power:GND #PWR038
 U 1 1 604AE05B
-P 8750 2250
-F 0 "#PWR038" H 8750 2000 50  0001 C CNN
-F 1 "GND" H 8755 2077 50  0000 C CNN
-F 2 "" H 8750 2250 50  0001 C CNN
-F 3 "" H 8750 2250 50  0001 C CNN
-	1    8750 2250
+P 9200 2250
+F 0 "#PWR038" H 9200 2000 50  0001 C CNN
+F 1 "GND" H 9205 2077 50  0000 C CNN
+F 2 "" H 9200 2250 50  0001 C CNN
+F 3 "" H 9200 2250 50  0001 C CNN
+	1    9200 2250
 	1    0    0    -1
 $EndComp
@@
 L Connector:Conn_01x06_Female J11
 U 1 1 60A01DDC
-P 10000 1450
-F 0 "J11" H 10028 1380 50  0000 L CNN
-F 1 "Conn_01x06_Female" H 10028 1335 50  0001 L CNN
-F 2 "" H 10000 1450 50  0001 C CNN
-F 3 "~" H 10000 1450 50  0001 C CNN
-	1    10000 1450
+P 10250 1450
+F 0 "J11" H 10278 1380 50  0000 L CNN
+F 1 "Conn_01x06_Female" H 10278 1335 50  0001 L CNN
+F 2 "" H 10250 1450 50  0001 C CNN
+F 3 "~" H 10250 1450 50  0001 C CNN
+	1    10250 1450
 	1    0    0    -1
 $EndComp
@@
 L Connector:Conn_01x06_Female J12
 U 1 1 60A03D75
-P 10000 2350
-F 0 "J12" H 10028 2280 50  0000 L CNN
-F 1 "Conn_01x06_Female" H 10028 2235 50  0001 L CNN
-F 2 "" H 10000 2350 50  0001 C CNN
-F 3 "~" H 10000 2350 50  0001 C CNN
-	1    10000 2350
-	1    0    0    -1
-$EndComp
-Wire Wire Line
-	9150 1350 9800 1350
-Wire Wire Line
-	9150 1450 9800 1450
-Wire Wire Line
-	9150 1550 9800 1550
-Wire Wire Line
-	9150 1650 9800 1650
-Wire Wire Line
-	9150 1750 9800 1750
-Wire Wire Line
-	9600 1250 9600 2150
-Wire Wire Line
-	9600 2150 9800 2150
+P 10250 2350
+F 0 "J12" H 10278 2280 50  0000 L CNN
+F 1 "Conn_01x06_Female" H 10278 2235 50  0001 L CNN
+F 2 "" H 10250 2350 50  0001 C CNN
+F 3 "~" H 10250 2350 50  0001 C CNN
+	1    10250 2350
+	1    0    0    -1
+$EndComp
+Wire Wire Line
+	9600 1350 10050 1350
+Wire Wire Line
+	9600 1450 10050 1450
+Wire Wire Line
+	9600 1550 10050 1550
+Wire Wire Line
+	9600 1650 10050 1650
+Wire Wire Line
+	9600 1750 10050 1750
+Wire Wire Line
+	9850 1250 9850 2150
+Wire Wire Line
+	9850 2150 10050 2150
 $Comp
 L power:+5V #PWR041
 U 1 1 60A3BA13
-P 9600 1050
-F 0 "#PWR041" H 9600 900 50  0001 C CNN
-F 1 "+5V" H 9615 1223 50  0000 C CNN
-F 2 "" H 9600 1050 50  0001 C CNN
-F 3 "" H 9600 1050 50  0001 C CNN
-	1    9600 1050
-	1    0    0    -1
-$EndComp
-Wire Wire Line
-	9800 1250 9600 1250
-Wire Wire Line
-	9600 1050 9600 1250
-Connection ~ 9600 1250
-Connection ~ 9800 1250
-Wire Wire Line
-	9800 1250 9850 1250
-Wire Wire Line
-	9150 1850 9500 1850
-Wire Wire Line
-	9500 1850 9500 2250
-Wire Wire Line
-	9500 2250 9800 2250
-Wire Wire Line
-	9150 1950 9400 1950
-Wire Wire Line
-	9400 1950 9400 2350
-Wire Wire Line
-	9400 2350 9800 2350
-Wire Wire Line
-	9150 2050 9150 2450
-Wire Wire Line
-	9150 2450 9800 2450
+P 9850 1050
+F 0 "#PWR041" H 9850 900 50  0001 C CNN
+F 1 "+5V" H 9865 1223 50  0000 C CNN
+F 2 "" H 9850 1050 50  0001 C CNN
+F 3 "" H 9850 1050 50  0001 C CNN
+	1    9850 1050
+	1    0    0    -1
+$EndComp
+Wire Wire Line
+	10050 1250 9850 1250
+Wire Wire Line
+	9850 1050 9850 1250
+Connection ~ 9850 1250
+Connection ~ 10050 1250
+Wire Wire Line
+	10050 1250 10100 1250
+Wire Wire Line
+	9600 1850 9750 1850
+Wire Wire Line
+	9750 1850 9750 2250
+Wire Wire Line
+	9750 2250 10050 2250
+Wire Wire Line
+	9600 1950 9650 1950
+Wire Wire Line
+	9650 1950 9650 2350
+Wire Wire Line
+	9650 2350 10050 2350
+Wire Wire Line
+	9600 2050 9400 2450
+Wire Wire Line
+	9400 2450 10050 2450
 Wire Wire Line
 	9800 2550 9300 2550
@@
 	9150 3600 9800 3600
 Wire Wire Line
-	9600 2150 9600 3100
+	9850 2150 9850 3100
 Wire Wire Line
 	9600 3100 9800 3100
-Connection ~ 9600 2150
+Connection ~ 9850 2150
 $Comp
 L Connector:Conn_01x06_Female J10
@@
 Wire Wire Line
 	9600 4750 9750 4750
-Connection ~ 9600 3100
 Wire Wire Line
 	9150 3700 9500 3700
@@
 Connection ~ 900  2950
 $Comp
-L Connector:Conn_01x07_Female J?
+L Connector:Conn_01x07_Female J14
 U 1 1 60962CDF
 P 2400 2950
-F 0 "J?" H 2292 2425 50  0000 C CNN
+F 0 "J14" H 2292 2425 50  0000 C CNN
 F 1 "Conn_01x07_Female" H 2292 2516 50  0000 C CNN
 F 2 "" H 2400 2950 50  0001 C CNN
@@
 Wire Wire Line
 	800  2950 900  2950
+$Comp
+L Transistor_Array:ULN2803A U6
+U 1 1 60418EE2
+P 9200 1550
+F 0 "U6" H 9200 2117 50  0000 C CNN
+F 1 "ULN2803A" H 9200 2026 50  0000 C CNN
+F 2 "Package_DIP:DIP-18_W7.62mm" H 9250 900 50  0001 L CNN
+F 3 "http://www.ti.com/lit/ds/symlink/uln2803a.pdf" H 9300 1350 50  0001 C CNN
+	1    9200 1550
+	1    0    0    -1
+$EndComp
+Wire Wire Line
+	8100 1650 8450 1650
+Wire Wire Line
+	8450 1650 8450 1750
+Wire Wire Line
+	8450 1750 8800 1750
+Wire Wire Line
+	8100 1550 8500 1550
+Wire Wire Line
+	8500 1550 8500 1850
+Wire Wire Line
+	8500 1850 8800 1850
+Wire Wire Line
+	8100 1450 8550 1450
+Wire Wire Line
+	8550 1450 8550 1950
+Wire Wire Line
+	8550 1950 8800 1950
+Wire Wire Line
+	8100 1350 8600 1350
+Wire Wire Line
+	8600 1350 8600 2050
+Wire Wire Line
+	8600 2050 8800 2050
+Wire Wire Line
+	8100 2050 8350 2050
+Wire Wire Line
+	8350 2050 8350 1600
+Wire Wire Line
+	8350 1600 8700 1600
+Wire Wire Line
+	8700 1600 8700 1650
+Wire Wire Line
+	8700 1650 8800 1650
+Wire Wire Line
+	8100 1950 8250 1950
+Wire Wire Line
+	8250 1950 8250 1500
+Wire Wire Line
+	8250 1500 8700 1500
+Wire Wire Line
+	8700 1500 8700 1550
+Wire Wire Line
+	8700 1550 8800 1550
+Wire Wire Line
+	8100 1850 8200 1850
+Wire Wire Line
+	8200 1850 8200 1400
+Wire Wire Line
+	8200 1400 8700 1400
+Wire Wire Line
+	8700 1400 8700 1450
+Wire Wire Line
+	8700 1450 8800 1450
+Wire Wire Line
+	8100 1750 8150 1750
+Wire Wire Line
+	8150 1750 8150 1300
+Wire Wire Line
+	8150 1300 8700 1300
+Wire Wire Line
+	8700 1300 8700 1350
+Wire Wire Line
+	8700 1350 8800 1350
 $EndSCHEMATC

Commit message: Auch die Bedruckung jetzt auf beiden Seiten, Platine jetzt komplett für Links und Rechts
Parts:
- added C? (x2): CP, symbol Device:CP
- added D1: 1N4004, Diode_THT:D_DO-41_SOD81_P10.16mm_Horizontal, symbol Diode:1N4004
- added D?: B40C1500A, symbol Device:D_Bridge_+AA-
- added D?: B140C1000A, Diodes_THT:Diode_Bridge_DIP-4_W7.62mm_P5.08mm, symbol Device:D_Bridge_+-AA
- added J15: 2604-1102, CONN_2604-1102_4_WAG, symbol WAGO:2604-1102
- added J?: Conn_01x02_Female, symbol Connector:Conn_01x02_Female
- added R7: 1k5, Resistors_THT:R_Axial_DIN0207_L6.3mm_D2.5mm_P7.62mm_Horizontal, symbol Device:R
- added R8: 10K, Resistors_THT:R_Axial_DIN0207_L6.3mm_D2.5mm_P7.62mm_Horizontal, symbol Device:R
- added U9: 6N136, Package_DIP:DIP-8_W7.62mm, symbol Isolator:6N136
- added U?: TSR_1-24120, Converter_DCDC:Converter_DCDC_TRACO_TSR-1_THT, symbol Regulator_Switching:TSR_1-24120
- added U?: TSR_1-2450, Converter_DCDC:Converter_DCDC_TRACO_TSR-1_THT, symbol Regulator_Switching:TSR_1-2450
Connections:
- wire segments 253 -> 297
- no-connect marks 12 -> 10
Other:
- note added: "DCC-Interface"

Commit message: Wago-Klemmen 250-140x verwendet
Parts:
- removed J11: Conn_01x06_Female, symbol Connector:Conn_01x06_Female
- removed J15: 2604-1102, CONN_2604-1102_4_WAG, symbol WAGO:2604-1102
- removed J3: Power, symbol Connector:Conn_01x02_Female
- removed J4: Weiche 1, symbol Connector:Conn_01x03_Female
- removed J5: Weiche 2, symbol Connector:Conn_01x03_Female
- removed J6: Weiche 3, symbol Connector:Conn_01x03_Female
- removed J7: Weiche 4, symbol Connector:Conn_01x03_Female
- removed J8: Weiche 5, symbol Connector:Conn_01x03_Female
- removed J9: Power Weiche, symbol Connector:Conn_01x02_Female
- removed J?: Conn_01x02_Female, symbol Connector:Conn_01x02_Female
- removed K1: HFD2_005-S-L2-D, HFD2_005-S-L2-D:HFD2005SL2D, symbol HFD2_005-S-L2-D:HFD2_005-S-L2-D
- added DS1001: DC-10SGWA, Kingbright-LED:DIPS750W80P254L2540H825Q20N, symbol Kingbright-LED:DC-10SGWA
- added J1, J2, J3, J4, J5: 250-1404, Wago:250-1404, symbol Wago:250-1404
- added J1001: Conn_01x02_Female, Pin_Headers:Pin_Header_Straight_1x02_Pitch2.54mm, symbol Connector:Conn_01x02_Female
- added J11: 250-1406, Wago:CONN_250-1406_WAG, symbol Wago:250-1406
- added J31, J41: 2604-1102, CONN_2604-1102_4_WAG, symbol Wago:2604-1102
- added JP11: Jumper, Pin_Headers:Pin_Header_Straight_1x02_Pitch2.54mm, symbol Device:Jumper
- added R7, R8: 1k, Resistors_THT:R_Array_SIP6, symbol Device:R_Network05
- C1: renamed from C?; value CP -> 2200µ/35V; footprint (none) -> Capacitors_THT:CP_Radial_D16.0mm_P7.50mm
- C2: renamed from C?; value CP -> 2200µF/35V; footprint (none) -> Capacitors_THT:CP_Radial_D16.0mm_P7.50mm
- D1: footprint Diode_THT:D_DO-41_SOD81_P10.16mm_Horizontal -> Diodes_THT:D_DO-15_P10.16mm_Horizontal
- D2: renamed from D?; footprint (none) -> Diodes_THT:Diode_Bridge_DIP-4_W7.62mm_P5.08mm
- J1003: renamed from J14; footprint (none) -> Pin_Headers:Pin_Header_Straight_1x07_Pitch2.54mm
- J12, J13: value Conn_01x06_Female -> Wago 250-1406; footprint (none) -> Wago:CONN_250-1406_WAG; symbol Connector:Conn_01x06_Female -> Wago:250-1406
- J14: renamed from J10; value Conn_01x06_Female -> Wago 250-1406; footprint (none) -> Wago:CONN_250-1406_WAG; symbol Connector:Conn_01x06_Female -> Wago:250-1406
- J22: renamed from J2; value RJ45_Shielded -> J22
- JP1: renamed from JP2; footprint Connectors:GS2 -> Pin_Headers:Pin_Header_Straight_1x02_Pitch2.54mm
- JP2: renamed from JP3; footprint Connectors:GS2 -> Pin_Headers:Pin_Header_Straight_1x02_Pitch2.54mm
- JP3: renamed from JP4; footprint Connectors:GS2 -> Pin_Headers:Pin_Header_Straight_1x02_Pitch2.54mm
- JP4: renamed from JP1; footprint (none) -> Pin_Headers:Pin_Header_Straight_1x02_Pitch2.54mm
- Shield1001: renamed from Shield1; footprint kicad-lib:MCP2515_CAN_MODULE_BY0-10 -> CAN-BUS-MODULE:MCP2515_CAN_MODULE_BY0-10
- U10, U11: renamed from U?; footprint Converter_DCDC:Converter_DCDC_TRACO_TSR-1_THT -> Converters_DCDC_ACDC:DCDC-Conv_TRACO_TSR-1
- gave numbers to parts that had none: 1
- renumbered C1 to C1001, C2 to C1002, C3 to C1003, J1 to J21, R7 to R1, R4 to R1007, R5 to R1008, R8 to R2, R6 to R3, R1 to R4, R3 to R5, R2 to R6, A1 to U1, U9 to U1001, U1 to U2, U2 to U3, U3 to U4, U4 to U5, U5 to U6, U6 to U7, U7 to U8, U8 to U9
Connections:
- wire segments 297 -> 342
Other:
- moved on the sheet: C1, C2, D2, D3, JP4, U10, U11, U3

Commit message: PCP weiterentwickelt
Parts:
- removed J21: RJ45_LED_Shielded, Connectors:RJ45_TRANSFO, symbol Connector:RJ45_LED_Shielded
- removed R3: 1K, Resistors_SMD:R_0603, symbol Device:R
- added J15: Wago 250-1406, Wago:CONN_250-1406_WAG, symbol Wago:250-1406
- added J23: J22, ASSMANN_WSW:A20042LPFS, symbol ASSMANN_WSW:A-20042-LP_FS
- added JP23: 12V CAN, Pin_Headers:Pin_Header_Straight_1x02_Pitch2.54mm, symbol Device:Jumper
- added JP41: DCC B, Pin_Headers:Pin_Header_Straight_1x02_Pitch2.54mm, symbol Jumper:Jumper_2_Open
- added JP42: DCC A, Pin_Headers:Pin_Header_Straight_1x02_Pitch2.54mm, symbol Jumper:Jumper_2_Open
- J22: footprint Connectors:RJ45_8 -> ASSMANN_WSW:A20042LPFS; symbol Connector:RJ45_Shielded -> ASSMANN_WSW:A-20042-LP_FS
- JP1: value JP3 -> Prog 1
- JP2: value JP1 -> Prog2
- JP3: value JP2 -> Prog3
- R4, R5, R6: footprint Resistors_SMD:R_0603 -> Resistors_THT:R_Axial_DIN0207_L6.3mm_D2.5mm_P7.62mm_Horizontal
- R7: renamed from R1007; footprint Resistors_SMD:R_0603 -> Resistors_THT:R_Axial_DIN0207_L6.3mm_D2.5mm_P7.62mm_Horizontal
- R8: renamed from R1008; footprint Resistors_SMD:R_0603 -> Resistors_THT:R_Axial_DIN0207_L6.3mm_D2.5mm_P7.62mm_Horizontal
- renumbered C1 to C10, C2 to C11, C1002 to C4, C1003 to C5, C1001 to C6, R8 to R10, R7 to R9
Connections:
- wire segments 342 -> 349
Other:
- moved on the sheet: C10, C11, C4, C5, C6, D1, D2, D3, DS1001, J1, J1001, J1003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

Commit message: Erster kompletter Entwurf der Platine
Parts:
- removed C10: 2200µ/35V, Capacitors_THT:CP_Radial_D16.0mm_P7.50mm, symbol Device:CP
- removed C11: 2200µF/35V, Capacitors_THT:CP_Radial_D16.0mm_P7.50mm, symbol Device:CP
- removed D2: B40C1500A, Diodes_THT:Diode_Bridge_DIP-4_W7.62mm_P5.08mm, symbol Device:D_Bridge_+AA-
- removed D3: B140C1000A, Diodes_THT:Diode_Bridge_DIP-4_W7.62mm_P5.08mm, symbol Device:D_Bridge_+-AA
- removed U11: TSR_1-2450, Converters_DCDC_ACDC:DCDC-Conv_TRACO_TSR-1, symbol Regulator_Switching:TSR_1-2450
- added D1001: DIODE, Diodes_THT:D_DO-15_P10.16mm_Horizontal, symbol pspice:DIODE
- added D1002: LED, LEDs:LED_D3.0mm, symbol Device:LED
- added R20: 470, Resistors_THT:R_Axial_DIN0207_L6.3mm_D2.5mm_P7.62mm_Horizontal, symbol Device:R
- J31: value 2604-1102 -> 12V DC
- U10: value TSR_1-24120 -> TSR_1-2450
Connections:
- net +12V: now also J31.1, J31.2, D1001.1 (K); no longer JP23.2
- net +5V: now also R20.2
- net GND: now also J31.3, J31.4, D1002.1 (K)
- net at U10.1 (Vin): now also JP23.2, D1001.2 (A)
- net at D1.2 (A), JP41.1 (A), U1001.3: now also J41.1, J41.2; no longer J41.3, J41.4
- net at JP42.1 (A), R1.2: now also J41.3, J41.4; no longer J41.1, J41.2
- new net: D1002.2 (A), R20.1
Other:
- moved on the sheet: J31, U10

Commit message: verbessert
Parts:
- removed J1001: Conn_01x02_Female, Pin_Headers:Pin_Header_Straight_1x02_Pitch2.54mm, symbol Connector:Conn_01x02_Female
- removed J1003: Conn_01x07_Female, Pin_Headers:Pin_Header_Straight_1x07_Pitch2.54mm, symbol Connector:Conn_01x07_Female
- added H1, H2, H3, H4: MountingHole, Mounting_Holes:MountingHole_3.2mm_M3, symbol Mechanical:MountingHole
Connections:
- net +5V: now also Shield1001.1 (VCC)
- net GND: now also Shield1001.2 (GND)
- net at U1.13 (D10): now also Shield1001.3 (CS)
- net at U1.14 (D11): now also Shield1001.5 (MOSI)
- net at U1.15 (D12): now also Shield1001.4 (MISO)
- net at U1.16 (D13): now also Shield1001.6 (SCK)
- net at U1.5 (D2): now also Shield1001.7 (INT)
- net at Shield1001.1.1 (J1-1): now also JP11.1
- net at Shield1001.1.2 (J1-2): now also JP11.2
Other:
- moved on the sheet: JP11, Shield1001
Changed lines of the file:
@@
 L CAN-BUS-MODULE-TJA1050:CAN-BUS_MODULE_TJA1050 Shield1001
 U 1 1 60585225
-P 2000 2650
-F 0 "Shield1001" H 1950 1975 50  0000 C CNN
-F 1 "CAN-BUS_MODULE_TJA1050" H 1950 1884 50  0000 C CNN
-F 2 "CAN-BUS-MODULE:MCP2515_CAN_MODULE_BY0-10" H 2000 2650 50  0001 C CIN
-F 3 "" H 2000 2650 50  0001 C CNN
-	1    2000 2650
+P 2200 2650
+F 0 "Shield1001" H 2150 1975 50  0000 C CNN
+F 1 "CAN-BUS_MODULE_TJA1050" H 2150 1884 50  0000 C CNN
+F 2 "CAN-BUS-MODULE:MCP2515_CAN_MODULE_BY0-10" H 2200 2650 50  0001 C CIN
+F 3 "" H 2200 2650 50  0001 C CNN
+	1    2200 2650
 	1    0    0    -1
 $EndComp
@@
 	2700 5000 2150 5000
 Wire Wire Line
-	1400 2850 1200 2850
+	1400 2850 1150 2850
 Wire Wire Line
 	1150 2850 1150 3550
 Wire Wire Line
-	1400 2750 1200 2750
+	1400 2750 1100 2750
 Wire Wire Line
 	1100 2750 1100 3600
 Wire Wire Line
 	4750 1750 3800 1750
-Connection ~ 1200 2850
-Wire Wire Line
-	1200 2850 1150 2850
-Connection ~ 1200 2750
-$Comp
-L Connector:Conn_01x07_Female J1003
-U 1 1 60962CDF
-P 2700 2750
-F 0 "J1003" H 2592 2225 50  0000 C CNN
-F 1 "Conn_01x07_Female" H 2592 2316 50  0000 C CNN
-F 2 "Pin_Headers:Pin_Header_Straight_1x07_Pitch2.54mm" H 2700 2750 50  0001 C CNN
-F 3 "~" H 2700 2750 50  0001 C CNN
-	1    2700 2750
-	-1   0    0    1
-$EndComp
-Wire Wire Line
-	1100 2750 1200 2750
 $Comp
 L Isolator:6N136 U1001
@@
 	1150 7200 1150 7100
 Connection ~ 1150 7100
-$Comp
-L Connector:Conn_01x02_Female J1001
-U 1 1 61A1EF28
-P 2100 2250
-F 0 "J1001" V 1946 2298 50  0000 L CNN
-F 1 "Conn_01x02_Female" V 2037 2298 50  0000 L CNN
-F 2 "Pin_Headers:Pin_Header_Straight_1x02_Pitch2.54mm" H 2100 2250 50  0001 C CNN
-F 3 "~" H 2100 2250 50  0001 C CNN
-	1    2100 2250
-	0    1    1    0
-$EndComp
-Wire Wire Line
-	1750 1900 1750 2050
-Wire Wire Line
-	1750 2050 2000 2050
-Wire Wire Line
-	2100 2050 2350 2050
-Wire Wire Line
-	2350 2050 2350 1900
+Wire Wire Line
+	1950 2100 1950 2250
+Wire Wire Line
+	1950 2250 2200 2250
+Wire Wire Line
+	2550 2250 2550 2100
 $Comp
 L Device:Jumper JP11
 U 1 1 61A202D7
-P 2050 1900
-F 0 "JP11" H 2050 2100 50  0000 C CNN
-F 1 "Jumper" H 2050 2073 50  0001 C CNN
-F 2 "Pin_Headers:Pin_Header_Straight_1x02_Pitch2.54mm" H 2050 1900 50  0001 C CNN
-F 3 "~" H 2050 1900 50  0001 C CNN
-	1    2050 1900
+P 2250 2100
+F 0 "JP11" H 2250 2300 50  0000 C CNN
+F 1 "Jumper" H 2250 2273 50  0001 C CNN
+F 2 "Pin_Headers:Pin_Header_Straight_1x02_Pitch2.54mm" H 2250 2100 50  0001 C CNN
+F 3 "~" H 2250 2100 50  0001 C CNN
+	1    2250 2100
 	1    0    0    -1
 $EndComp
@@
 	3450 7350 2850 7350
 Connection ~ 2850 7350
+Wire Wire Line
+	2300 2250 2550 2250
+$Comp
+L Mechanical:MountingHole H1
+U 1 1 622C717E
+P 10250 6000
+F 0 "H1" H 10350 6046 50  0000 L CNN
+F 1 "MountingHole" H 10350 5955 50  0000 L CNN
+F 2 "Mounting_Holes:MountingHole_3.2mm_M3" H 10250 6000 50  0001 C CNN
+F 3 "~" H 10250 6000 50  0001 C CNN
+	1    10250 6000
+	1    0    0    -1
+$EndComp
+$Comp
+L Mechanical:MountingHole H2
+U 1 1 622C9821
+P 10250 6250
+F 0 "H2" H 10350 6296 50  0000 L CNN
+F 1 "MountingHole" H 10350 6205 50  0000 L CNN
+F 2 "Mounting_Holes:MountingHole_3.2mm_M3" H 10250 6250 50  0001 C CNN
+F 3 "~" H 10250 6250 50  0001 C CNN
+	1    10250 6250
+	1    0    0    -1
+$EndComp
+$Comp
+L Mechanical:MountingHole H4
+U 1 1 62312DA2
+P 9950 6250
+F 0 "H4" H 10050 6296 50  0000 L CNN
+F 1 "MountingHole" H 10050 6205 50  0000 L CNN
+F 2 "Mounting_Holes:MountingHole_3.2mm_M3" H 9950 6250 50  0001 C CNN
+F 3 "~" H 9950 6250 50  0001 C CNN
+	1    9950 6250
+	1    0    0    -1
+$EndComp
+$Comp
+L Mechanical:MountingHole H3
+U 1 1 62380421
+P 9950 5900
+F 0 "H3" H 10050 5946 50  0000 L CNN
+F 1 "MountingHole" H 10050 5855 50  0000 L CNN
+F 2 "Mounting_Holes:MountingHole_3.2mm_M3" H 9950 5900 50  0001 C CNN
+F 3 "~" H 9950 5900 50  0001 C CNN
+	1    9950 5900
+	1    0    0    -1
+$EndComp
 $EndSCHEMATC
