File: doc/kicad/CAN-BUS-Weichendecoder-Weiche-small/CAN-BUS-Weichendecoder-Weiche-small.kicad_pcb (KiCad board)
At the start: 2 copper layers, 151.1 x 88.9 mm, 39 parts, among them J1 250-1404, J1001 I²C, J1002 Conn_01x16_Male, J2 250-1404, J22 J22, J23 J22, J3 250-1404, J31 12V DC, J4 250-1404, J41 2604-1102, J5 250-1404, U1 Arduino_Nano, U10 TSR_1-2450, U1001 6N136, U2 ULN2803A, U3 ULN2803A

Commit message: Aktuellen zwischenstand gesichert
Parts:
- removed J1, J2, J3, J4, J5: 250-1404, Wago:250-1404
- added H1: MountingHole, Mounting_Holes:MountingHole_3.2mm_M3, F.Cu at (168.9, 47.0)
- added H2: MountingHole, Mounting_Holes:MountingHole_3.2mm_M3, F.Cu at (168.9, 108.0)
- added H3: MountingHole, Mounting_Holes:MountingHole_3.2mm_M3, F.Cu at (54.6, 109.2)
- added H4: MountingHole, Mounting_Holes:MountingHole_3.2mm_M3, F.Cu at (50.8, 41.9)
- J1002: footprint Connectors:he10-16d -> Connectors_Samtec:SL-116-X-XX_1x16
- JP11: value Jumper -> CAN-Term
- moved JP4 70.0 mm to (96.5, 54.6)
- moved J1002 26.1 mm to (97.8, 45.7), turned to 90 degrees
- moved U3 12.7 mm to (129.5, 58.4)
- moved JP23 6.35 mm to (55.9, 74.9)
- moved J1001 3.81 mm to (119.4, 101.6)
- moved R7 3.59 mm to (116.8, 95.2)
- moved R8 3.59 mm to (116.8, 91.4)
- moved JP1 2.84 mm to (144.8, 99.1)
- moved JP3 2.84 mm to (144.8, 95.2)
- moved R5 2.84 mm to (132.1, 99.1)
- moved JP2 2.84 mm to (144.8, 91.4)
- moved R4 2.84 mm to (132.1, 91.4)
- moved R6 2.54 mm to (128.3, 95.2)
- moved JP11 1.80 mm to (92.7, 96.5)
- moved CAN-Bus1001 1.27 mm to (45.7, 92.7)
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- renumbered J23 to CAN-Bus1001, J22 to CAN-Bus1002
Connections:
- J1002 pad 1: Net-(J1-Pad3) -> +12V
- J1002 pad 11: GND -> Net-(J1002-Pad11)
- J1002 pad 12: +12V -> Net-(J1002-Pad12)
- J1002 pad 13: GND -> (no net)
- J1002 pad 14: +12V -> (no net)
- J1002 pad 16: +12V -> GND
- J1002 pad 2: Net-(J1-Pad2) -> +12V
- U2 pad 11: Net-(J1002-Pad7) -> Net-(J1002-Pad10)
- U2 pad 12: Net-(J1002-Pad8) -> Net-(J1002-Pad9)
- U2 pad 13: Net-(J1002-Pad5) -> Net-(J1002-Pad8)
- U2 pad 14: Net-(J1002-Pad6) -> Net-(J1002-Pad7)
- U2 pad 15: Net-(J1002-Pad3) -> Net-(J1002-Pad6)
- U2 pad 16: Net-(J1002-Pad4) -> Net-(J1002-Pad5)
- U2 pad 17: Net-(J1-Pad3) -> Net-(J1002-Pad4)
- U2 pad 18: Net-(J1-Pad2) -> Net-(J1002-Pad3)
- U3 pad 17: Net-(J1002-Pad9) -> Net-(J1002-Pad12)
- U3 pad 18: Net-(J1002-Pad10) -> Net-(J1002-Pad11)
Routing:
- net GND: track 552.4 -> 451.2 mm
- net +12V: track 177.8 -> 99.9 mm
- net Net-(J1002-Pad7): track 58.8 -> 5.08 mm
- net Net-(J1002-Pad9): track 58.3 -> 5.08 mm
- net Net-(J1002-Pad10): track 56.5 -> 5.08 mm
- net Net-(J1002-Pad8): track 56.1 -> 5.08 mm
- net Net-(J1-Pad2): track 37.1 -> 0.00 mm
- net Net-(J1002-Pad6): track 42.2 -> 5.08 mm
- net Net-(J1002-Pad5): track 41.8 -> 5.08 mm
- net Net-(J1-Pad3): track 31.3 -> 0.00 mm
- net Net-(J1002-Pad4): track 30.1 -> 5.08 mm
- net Net-(J1002-Pad3): track 26.5 -> 5.08 mm
- net Net-(DS1001-Pad9): track 70.5 -> 81.7 mm
- net Net-(DS1001-Pad10): track 69.2 -> 79.7 mm
- net +5V: track 156.9 -> 146.8 mm
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Other:
- board size 151.1 x 88.9 mm -> 151.1 x 87.6 mm
