File: doc/kicad/CAN-BUS-Weichendecoder-Weiche-small/CAN-BUS-Weichendecoder-Weiche-small.sch (KiCad schematic (older format))
At the start: 39 parts, among them J1 250-1404, J1001 I²C, J1002 Conn_01x16_Male, J2 250-1404, J3 250-1404, J31 12V DC, J4 250-1404, J41 2604-1102, J5 250-1404, U1 Arduino_Nano, U10 TSR_1-2450, U1001 6N136, U2 ULN2803A, U3 ULN2803A

Commit message: Aktuellen zwischenstand gesichert
Parts:
- removed J1, J2, J3, J4, J5: 250-1404, Wago:250-1404, symbol Wago:250-1404
- added H1, H2, H3, H4: MountingHole, Mounting_Holes:MountingHole_3.2mm_M3, symbol Mechanical:MountingHole
- J1002: footprint Connectors:he10-16d -> Connectors_Samtec:SL-116-X-XX_1x16
- renumbered CAN-Bus to CAN-Bus1001, CAN-Bus to CAN-Bus1002
Connections:
- wire segments 318 -> 241
Other:
- moved on the sheet: J1002
