File: doc/kicad/Belegmelder_Neustadt/Belegmelder_Neustadt.sch (KiCad schematic (older format))
At the start: 17 parts, among them T1 BC547

Commit message: Aufgeräumt
Parts:
- C1: value 100nF -> 100nF (MKS); footprint (none) -> Capacitors_SMD:C_2220
- C2: renamed from C?; value C -> 10nF; footprint (none) -> Capacitors_SMD:C_0805
- C3: footprint (none) -> Capacitors_SMD:CP_Elec_4x5.3
- D1, D2, D3: footprint (none) -> Diodes_SMD:D_SOD-323F
- D4: renamed from D?; footprint (none) -> LEDs:LED_0805
- L1: footprint (none) -> Talema:AS-1xx
- R1, R2, R3, R4, R5, R6, R7: footprint (none) -> Resistors_SMD:R_0805
- T1: value BC547 -> BC547/BC847C; footprint Package_TO_SOT_THT:TO-92_Inline -> TO_SOT_Packages_SMD:SOT-23
- T2: renamed from Q?; footprint Package_TO_SOT_THT:TO-92_Inline -> TO_SOT_Packages_SMD:SOT-23
Changed lines of the file:
@@
 F 0 "L1" H 2656 1854 50  0000 R CNN
 F 1 "Talema AS100" V 2850 2150 50  0000 R CNN
-F 2 "" H 2700 1900 50  0001 C CNN
+F 2 "Talema:AS-1xx" H 2700 1900 50  0001 C CNN
 F 3 "~" H 2700 1900 50  0001 C CNN
 	1    2700 1900
@@
 F 0 "R1" H 3470 1446 50  0000 L CNN
 F 1 "3k3" H 3470 1355 50  0000 L CNN
-F 2 "" V 3330 1400 50  0001 C CNN
+F 2 "Resistors_SMD:R_0805" V 3330 1400 50  0001 C CNN
 F 3 "~" H 3400 1400 50  0001 C CNN
 	1    3400 1400
@@
 F 0 "R2" H 3470 2396 50  0000 L CNN
 F 1 "560" H 3470 2305 50  0000 L CNN
-F 2 "" V 3330 2350 50  0001 C CNN
+F 2 "Resistors_SMD:R_0805" V 3330 2350 50  0001 C CNN
 F 3 "~" H 3400 2350 50  0001 C CNN
 	1    3400 2350
@@
 F 0 "D1" V 3446 2570 50  0000 R CNN
 F 1 "1N4148" V 3355 2570 50  0000 R CNN
-F 2 "" H 3400 2650 50  0001 C CNN
+F 2 "Diodes_SMD:D_SOD-323F" H 3400 2650 50  0001 C CNN
 F 3 "~" H 3400 2650 50  0001 C CNN
 	1    3400 2650
@@
 $EndComp
 $Comp
-L power:GND #PWR?
+L power:GND #PWR0101
 U 1 1 616BB44F
 P 3400 3050
-F 0 "#PWR?" H 3400 2800 50  0001 C CNN
+F 0 "#PWR0101" H 3400 2800 50  0001 C CNN
 F 1 "GND" H 3405 2877 50  0000 C CNN
 F 2 "" H 3400 3050 50  0001 C CNN
@@
 F 0 "R3" V 3843 2000 50  0000 C CNN
 F 1 "220k" V 3934 2000 50  0000 C CNN
-F 2 "" V 3980 2000 50  0001 C CNN
+F 2 "Resistors_SMD:R_0805" V 3980 2000 50  0001 C CNN
 F 3 "~" H 4050 2000 50  0001 C CNN
 	1    4050 2000
@@
 $EndComp
 $Comp
-L Device:C C?
+L Device:C C2
 U 1 1 616BC7F1
 P 4050 2300
-F 0 "C?" H 4165 2346 50  0000 L CNN
-F 1 "C" H 4165 2255 50  0000 L CNN
-F 2 "" H 4088 2150 50  0001 C CNN
+F 0 "C2" V 3800 2300 50  0000 L CNN
+F 1 "10nF" V 3900 2250 50  0000 L CNN
+F 2 "Capacitors_SMD:C_0805" H 4088 2150 50  0001 C CNN
 F 3 "~" H 4050 2300 50  0001 C CNN
 	1    4050 2300
@@
 P 3000 1900
 F 0 "C1" H 2885 1854 50  0000 R CNN
-F 1 "100nF" H 2885 1945 50  0000 R CNN
-F 2 "" H 3038 1750 50  0001 C CNN
+F 1 "100nF (MKS)" H 2885 1945 50  0000 R CNN
+F 2 "Capacitors_SMD:C_2220" H 3038 1750 50  0001 C CNN
 F 3 "~" H 3000 1900 50  0001 C CNN
 	1    3000 1900
@@
 F 0 "D2" V 4254 2730 50  0000 L CNN
 F 1 "1N4148" V 4345 2730 50  0000 L CNN
-F 2 "" H 4300 2650 50  0001 C CNN
+F 2 "Diodes_SMD:D_SOD-323F" H 4300 2650 50  0001 C CNN
 F 3 "~" H 4300 2650 50  0001 C CNN
 	1    4300 2650
@@
 P 4650 2000
 F 0 "T1" H 4841 2046 50  0000 L CNN
-F 1 "BC547" H 4841 1955 50  0000 L CNN
-F 2 "Package_TO_SOT_THT:TO-92_Inline" H 4850 1925 50  0001 L CIN
+F 1 "BC547/BC847C" H 4841 1955 50  0000 L CNN
+F 2 "TO_SOT_Packages_SMD:SOT-23" H 4850 1925 50  0001 L CIN
 F 3 "https://www.onsemi.com/pub/Collateral/BC550-D.pdf" H 4650 2000 50  0001 L CNN
 	1    4650 2000
@@
 F 0 "R4" H 4820 1446 50  0000 L CNN
 F 1 "3k3" H 4820 1355 50  0000 L CNN
-F 2 "" V 4680 1400 50  0001 C CNN
+F 2 "Resistors_SMD:R_0805" V 4680 1400 50  0001 C CNN
 F 3 "~" H 4750 1400 50  0001 C CNN
 	1    4750 1400
@@
 F 0 "D3" H 5050 1533 50  0000 C CNN
 F 1 "1N4148" H 5050 1624 50  0000 C CNN
-F 2 "" H 5050 1750 50  0001 C CNN
+F 2 "Diodes_SMD:D_SOD-323F" H 5050 1750 50  0001 C CNN
 F 3 "~" H 5050 1750 50  0001 C CNN
 	1    5050 1750
@@
 Wire Wire Line
 	4750 1750 4750 1800
+$Comp
+L Device:R R5
+U 1 1 616C8704
+P 5800 2200
+F 0 "R5" H 5870 2246 50  0000 L CNN
+F 1 "220k" H 5870 2155 50  0000 L CNN
+F 2 "Resistors_SMD:R_0805" V 5730 2200 50  0001 C CNN
+F 3 "~" H 5800 2200 50  0001 C CNN
+	1    5800 2200
+	1    0    0    -1
+$EndComp
+Wire Wire Line
+	5200 1750 5300 1750
+Wire Wire Line
+	5300 1750 5300 2300
+Wire Wire Line
+	5300 1750 5800 1750
+Wire Wire Line
+	5800 1750 5800 2050
+Connection ~ 5300 1750
+Wire Wire Line
+	5300 2600 5300 2900
+Wire Wire Line
+	5300 2900 4750 2900
+Connection ~ 4750 2900
+Wire Wire Line
+	5800 2350 5800 2900
+Wire Wire Line
+	5800 2900 5300 2900
+Connection ~ 5300 2900
+$Comp
+L Transistor_FET:BS170 T2
+U 1 1 616CA598
+P 6100 1750
+F 0 "T2" H 6304 1796 50  0000 L CNN
+F 1 "BS170" H 6304 1705 50  0000 L CNN
+F 2 "TO_SOT_Packages_SMD:SOT-23" H 6300 1675 50  0001 L CIN
+F 3 "https://www.onsemi.com/pub/Collateral/BS170-D.PDF" H 6100 1750 50  0001 L CNN
+	1    6100 1750
+	1    0    0    -1
+$EndComp
+Wire Wire Line
+	6200 1950 6200 2900
+Wire Wire Line
+	6200 2900 5800 2900
+Connection ~ 5800 2900
+Wire Wire Line
+	5800 1750 5900 1750
+Connection ~ 5800 1750
+$Comp
+L power:+5P #PWR0102
+U 1 1 616CB964
+P 3400 800
+F 0 "#PWR0102" H 3400 650 50  0001 C CNN
+F 1 "+5P" H 3415 973 50  0000 C CNN
+F 2 "" H 3400 800 50  0001 C CNN
+F 3 "" H 3400 800 50  0001 C CNN
+	1    3400 800
+	1    0    0    -1
+$EndComp
+Wire Wire Line
+	3400 800  3400 1000
+Connection ~ 3400 1000
+Wire Wire Line
+	6200 1550 6200 1400
+Wire Wire Line
+	6200 1400 6900 1400
+$Comp
+L Device:R R7
+U 1 1 616DC4CF
+P 6900 1200
+F 0 "R7" H 6970 1246 50  0000 L CNN
+F 1 "10k" H 6970 1155 50  0000 L CNN
+F 2 "Resistors_SMD:R_0805" V 6830 1200 50  0001 C CNN
+F 3 "~" H 6900 1200 50  0001 C CNN
+	1    6900 1200
+	1    0    0    -1
+$EndComp
+Wire Wire Line
+	6900 1350 6900 1400
+Wire Wire Line
+	4750 1000 6900 1000
+Wire Wire Line
+	6900 1000 6900 1050
+Connection ~ 4750 1000
+Wire Wire Line
+	6900 1400 7600 1400
+Connection ~ 6900 1400
+$Comp
+L Device:R R6
+U 1 1 616DEE8D
+P 6900 1850
+F 0 "R6" H 6970 1896 50  0000 L CNN
+F 1 "2k2" H 6970 1805 50  0000 L CNN
+F 2 "Resistors_SMD:R_0805" V 6830 1850 50  0001 C CNN
+F 3 "~" H 6900 1850 50  0001 C CNN
+	1    6900 1850
+	1    0    0    -1
+$EndComp
+$Comp
+L Device:LED D4
+U 1 1 616DF90F
+P 6900 2350
+F 0 "D4" V 6939 2232 50  0000 R CNN
+F 1 "LED" V 6848 2232 50  0000 R CNN
+F 2 "LEDs:LED_0805" H 6900 2350 50  0001 C CNN
+F 3 "~" H 6900 2350 50  0001 C CNN
+	1    6900 2350
+	0    -1   -1   0
+$EndComp
+Wire Wire Line
+	6900 1400 6900 1700
+Wire Wire Line
+	6900 2000 6900 2200
+Wire Wire Line
+	6900 2500 6900 2900
+Wire Wire Line
+	6900 2900 6200 2900
+Connection ~ 6200 2900
 $Comp
 L Device:CP C3
@@
 F 0 "C3" H 5418 2496 50  0000 L CNN
 F 1 "1µF/16V" H 5418 2405 50  0000 L CNN
-F 2 "" H 5338 2300 50  0001 C CNN
+F 2 "Capacitors_SMD:CP_Elec_4x5.3" H 5338 2300 50  0001 C CNN
 F 3 "~" H 5300 2450 50  0001 C CNN
 	1    5300 2450
 	1    0    0    -1
 $EndComp
-$Comp
-L Device:R R5
-U 1 1 616C8704
-P 5800 2200
-F 0 "R5" H 5870 2246 50  0000 L CNN
-F 1 "220k" H 5870 2155 50  0000 L CNN
-F 2 "" V 5730 2200 50  0001 C CNN
-F 3 "~" H 5800 2200 50  0001 C CNN
-	1    5800 2200
-	1    0    0    -1
-$EndComp
-Wire Wire Line
-	5200 1750 5300 1750
-Wire Wire Line
-	5300 1750 5300 2300
-Wire Wire Line
-	5300 1750 5800 1750
-Wire Wire Line
-	5800 1750 5800 2050
-Connection ~ 5300 1750
-Wire Wire Line
-	5300 2600 5300 2900
-Wire Wire Line
-	5300 2900 4750 2900
-Connection ~ 4750 2900
-Wire Wire Line
-	5800 2350 5800 2900
-Wire Wire Line
-	5800 2900 5300 2900
-Connection ~ 5300 2900
-$Comp
-L Transistor_FET:BS170 Q?
-U 1 1 616CA598
-P 6100 1750
-F 0 "Q?" H 6304 1796 50  0000 L CNN
-F 1 "BS170" H 6304 1705 50  0000 L CNN
-F 2 "Package_TO_SOT_THT:TO-92_Inline" H 6300 1675 50  0001 L CIN
-F 3 "https://www.onsemi.com/pub/Collateral/BS170-D.PDF" H 6100 1750 50  0001 L CNN
-	1    6100 1750
-	1    0    0    -1
-$EndComp
-Wire Wire Line
-	6200 1950 6200 2900
-Wire Wire Line
-	6200 2900 5800 2900
-Connection ~ 5800 2900
-Wire Wire Line
-	5800 1750 5900 1750
-Connection ~ 5800 1750
-$Comp
-L power:+5P #PWR?
-U 1 1 616CB964
-P 3400 800
-F 0 "#PWR?" H 3400 650 50  0001 C CNN
-F 1 "+5P" H 3415 973 50  0000 C CNN
-F 2 "" H 3400 800 50  0001 C CNN
-F 3 "" H 3400 800 50  0001 C CNN
-	1    3400 800
-	1    0    0    -1
-$EndComp
-Wire Wire Line
-	3400 800  3400 1000
-Connection ~ 3400 1000
-Wire Wire Line
-	6200 1550 6200 1400
-Wire Wire Line
-	6200 1400 6900 1400
-$Comp
-L Device:R R7
-U 1 1 616DC4CF
-P 6900 1200
-F 0 "R7" H 6970 1246 50  0000 L CNN
-F 1 "10k" H 6970 1155 50  0000 L CNN
-F 2 "" V 6830 1200 50  0001 C CNN
-F 3 "~" H 6900 1200 50  0001 C CNN
-	1    6900 1200
-	1    0    0    -1
-$EndComp
-Wire Wire Line
-	6900 1350 6900 1400
-Wire Wire Line
-	4750 1000 6900 1000
-Wire Wire Line
-	6900 1000 6900 1050
-Connection ~ 4750 1000
-Wire Wire Line
-	6900 1400 7600 1400
-Connection ~ 6900 1400
-$Comp
-L Device:R R6
-U 1 1 616DEE8D
-P 6900 1850
-F 0 "R6" H 6970 1896 50  0000 L CNN
-F 1 "2k2" H 6970 1805 50  0000 L CNN
-F 2 "" V 6830 1850 50  0001 C CNN
-F 3 "~" H 6900 1850 50  0001 C CNN
-	1    6900 1850
-	1    0    0    -1
-$EndComp
-$Comp
-L Device:LED D?
-U 1 1 616DF90F
-P 6900 2350
-F 0 "D?" V 6939 2232 50  0000 R CNN
-F 1 "LED" V 6848 2232 50  0000 R CNN
-F 2 "" H 6900 2350 50  0001 C CNN
-F 3 "~" H 6900 2350 50  0001 C CNN
-	1    6900 2350
-	0    -1   -1   0
-$EndComp
-Wire Wire Line
-	6900 1400 6900 1700
-Wire Wire Line
-	6900 2000 6900 2200
-Wire Wire Line
-	6900 2500 6900 2900
-Wire Wire Line
-	6900 2900 6200 2900
-Connection ~ 6200 2900
 $EndSCHEMATC
