File: doc/kicad/CAN-BUS-Weichendecoder-Signal/CAN-BUS-Weichendecoder-Signal.kicad_pcb (KiCad board)
At the start: 2 copper layers, 151.1 x 124.5 mm, 24 parts, among them J1 Conn_01x04_Male, J1001 Wago 250-1406, J11 250-1406, J12 Wago 250-1406, J13 Wago 250-1406, J14 Wago 250-1406, J15 Wago 250-1406, U1 PCF8574, U2 PCF8574, U3 PCF8574, U4 PCF8574, U5 ULN2803A, U6 ULN2803A, U7 ULN2803A, U8 ULN2803A

Commit message: Aufgeräumt
Parts:
- added J21: Conn_01x06, Connectors_IDC:IDC-Header_2x03_P2.54mm_Vertical, B.Cu at (86.4, 162.6)
- added J22: Conn_01x06, Connectors_IDC:IDC-Header_2x03_P2.54mm_Vertical, B.Cu at (106.7, 162.6)
Routing:
- net +5V: track 315.6 -> 370.9 mm
- net Net-(J11-Pad6): track 17.7 -> 35.2 mm
- net Net-(J12-Pad6): track 19.8 -> 37.2 mm
- net Net-(J12-Pad4): track 22.1 -> 37.4 mm
- net Net-(J11-Pad4): track 17.7 -> 31.6 mm
- net Net-(J12-Pad3): track 15.9 -> 29.3 mm
- net Net-(J11-Pad3): track 12.7 -> 23.9 mm
- net Net-(J11-Pad5): track 12.7 -> 22.1 mm
- net Net-(J12-Pad5): track 14.8 -> 24.2 mm
- net Net-(J12-Pad2): track 20.9 -> 29.9 mm
- net Net-(J11-Pad2): track 17.7 -> 25.8 mm
- net GND: track 199.0 -> 197.6 mm
- net Net-(JP1-Pad2): track 114.7 -> 114.1 mm
Other:
- net class Default removed
- net class Power removed
