File: doc/kicad/CAN-BUS-Weichendecoder-Signal/CAN-BUS-Weichendecoder-Signal.sch (KiCad schematic (older format))
At the start: 24 parts, among them J1 Conn_01x04_Male, J1001 Wago 250-1406, J11 250-1406, J12 Wago 250-1406, J13 Wago 250-1406, J14 Wago 250-1406, J15 Wago 250-1406, U1 PCF8574, U2 PCF8574, U3 PCF8574, U4 PCF8574, U5 ULN2803A, U6 ULN2803A, U7 ULN2803A, U8 ULN2803A

Commit message: Aufgeräumt
Parts:
- added J21, J22: Conn_01x06, Connectors_IDC:IDC-Header_2x03_P2.54mm_Vertical, symbol Connector_Generic:Conn_01x06
Connections:
- net +5V: now also J21.4 (Pin_4), J22.4 (Pin_4)
- net at J11.2, U5.11 (O8): now also J21.5 (Pin_5)
- net at J11.3, U5.12 (O7): now also J21.6 (Pin_6)
- net at J11.4, U5.13 (O6): now also J21.3 (Pin_3)
- net at J11.5, U5.14 (O5): now also J21.1 (Pin_1)
- net at J11.6, U5.15 (O4): now also J21.2 (Pin_2)
- net at J12.2, U5.16 (O3): now also J22.5 (Pin_5)
- net at J12.3, U5.17 (O2): now also J22.6 (Pin_6)
- net at J12.4, U5.18 (O1): now also J22.3 (Pin_3)
- net at J12.5, U6.11 (O8): now also J22.1 (Pin_1)
- net at J12.6, U6.12 (O7): now also J22.2 (Pin_2)
- no-connect marks 7 -> 10
Other:
- moved on the sheet: J12
