File: doc/kicad/Weichensimulator-45links/Weichensimulator-45links.kicad_sch (KiCad schematic)
At the start: 9 parts, among them J1 Conn_01x02_Male, J2 Power, J3 Conn_01x02_Male, K1 HFD2_005-S-L2-D

Commit message: Kosmetik
Parts:
- removed K1: HFD2_005-S-L2-D, HFD2005SL2D, symbol HFD2_005-S-L2-D:HFD2_005-S-L2-D
- added K1: HFD2_005-S-L2-D, HFD2005SL2D, symbol HongFa:HFD2_005-S-L2-D
Connections:
- net +5V: now also K1.1 (+SET), K1.2 (+RESET)
- net GND: now also K1.4 (COM_1)
- net at D2.1 (K): now also K1.8 (NO_1)
- net at D3.1 (K): now also K1.6 (NC_1)
- net at J1.1 (Pin_1): now also K1.15 (-RESET)
- net at J1.2 (Pin_2): now also K1.16 (-SET)
- no-connect marks 0 -> 3
Changed lines of the file:
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@@
   (junction (at 114.3 58.42) (diameter 0) (color 0 0 0 0)
   )
+  (no_connect (at 171.45 85.09))
+  (no_connect (at 171.45 87.63))
+  (no_connect (at 171.45 90.17))
   (wire (pts (xy 171.45 82.55) (xy 176.53 82.55))
     (stroke (width 0) (type default) (color 0 0 0 0))
@@
   )
   (wire (pts (xy 104.14 111.76) (xy 109.22 111.76))
+    (stroke (width 0) (type default) (color 0 0 0 0))
+  )
+  (wire (pts (xy 137.795 85.09) (xy 138.43 85.09))
     (stroke (width 0) (type default) (color 0 0 0 0))
   )
@@
     (pin "1")
   )
-  (symbol (lib_id "HFD2_005-S-L2-D:HFD2_005-S-L2-D") (at 138.43 80.01 0) (unit 1)
-    (in_bom yes) (on_board yes)
-    (property "Reference" "K1" (id 0) (at 154.94 73.279 0))
-    (property "Value" "HFD2_005-S-L2-D" (id 1) (at 154.94 75.5904 0))
+  (symbol (lib_id "power:GND") (at 137.795 85.09 270) (unit 1)
+    (in_bom yes) (on_board yes)
+    (property "Reference" "#PWR0102" (id 0) (at 131.445 85.09 0)
+      (effects (font (size 1.27 1.27)) hide)
+    )
+    (property "Value" "GND" (id 1) (at 134.5438 85.217 90)
+      (effects (font (size 1.27 1.27)) (justify right))
+    )
+    (property "Footprint" "" (id 2) (at 137.795 85.09 0)
+      (effects (font (size 1.27 1.27)) hide)
+    )
+    (property "Datasheet" "" (id 3) (at 137.795 85.09 0)
+      (effects (font (size 1.27 1.27)) hide)
+    )
+    (pin "1")
+  )
+  (symbol (lib_id "Connector:Conn_01x02_Male") (at 181.61 82.55 180) (unit 1)
+    (in_bom yes) (on_board yes)
+    (property "Reference" "J1" (id 0) (at 182.3212 80.7212 0)
+      (effects (font (size 1.27 1.27)) (justify right))
+    )
+    (property "Value" "Conn_01x02_Male" (id 1) (at 178.8668 84.836 0)
+      (effects (font (size 1.27 1.27)) hide)
+    )
+    (property "Footprint" "Pin_Headers:Pin_Header_Angled_1x02_Pitch2.54mm" (id 2) (at 181.61 82.55 0)
+      (effects (font (size 1.27 1.27)) hide)
+    )
+    (property "Datasheet" "~" (id 3) (at 181.61 82.55 0)
+      (effects (font (size 1.27 1.27)) hide)
+    )
+    (pin "1")
+    (pin "2")
+  )
+  (symbol (lib_id "Connector:Conn_01x02_Male") (at 99.06 97.79 0) (unit 1)
+    (in_bom yes) (on_board yes)
+    (property "Reference" "J2" (id 0) (at 101.8032 93.1926 0))
+    (property "Value" "Power" (id 1) (at 101.6 102.87 0))
+    (property "Footprint" "Pin_Headers:Pin_Header_Angled_1x02_Pitch2.54mm" (id 2) (at 99.06 97.79 0)
+      (effects (font (size 1.27 1.27)) hide)
+    )
+    (property "Datasheet" "~" (id 3) (at 99.06 97.79 0)
+      (effects (font (size 1.27 1.27)) hide)
+    )
+    (pin "1")
+    (pin "2")
+  )
+  (symbol (lib_id "power:+5V") (at 121.92 97.79 0) (unit 1)
+    (in_bom yes) (on_board yes)
+    (property "Reference" "#PWR0103" (id 0) (at 121.92 101.6 0)
+      (effects (font (size 1.27 1.27)) hide)
+    )
+    (property "Value" "+5V" (id 1) (at 122.301 93.3958 0))
+    (property "Footprint" "" (id 2) (at 121.92 97.79 0)
+      (effects (font (size 1.27 1.27)) hide)
+    )
+    (property "Datasheet" "" (id 3) (at 121.92 97.79 0)
+      (effects (font (size 1.27 1.27)) hide)
+    )
+    (pin "1")
+  )
+  (symbol (lib_id "power:GND") (at 121.92 100.33 0) (unit 1)
+    (in_bom yes) (on_board yes)
+    (property "Reference" "#PWR0104" (id 0) (at 121.92 106.68 0)
+      (effects (font (size 1.27 1.27)) hide)
+    )
+    (property "Value" "GND" (id 1) (at 122.047 104.7242 0))
+    (property "Footprint" "" (id 2) (at 121.92 100.33 0)
+      (effects (font (size 1.27 1.27)) hide)
+    )
+    (property "Datasheet" "" (id 3) (at 121.92 100.33 0)
+      (effects (font (size 1.27 1.27)) hide)
+    )
+    (pin "1")
+  )
+  (symbol (lib_id "Connector:Conn_01x02_Male") (at 99.06 109.22 0) (unit 1)
+    (in_bom yes) (on_board yes)
+    (property "Reference" "J3" (id 0) (at 101.8032 106.9594 0))
+    (property "Value" "Conn_01x02_Male" (id 1) (at 101.8032 106.934 0)
+      (effects (font (size 1.27 1.27)) hide)
+    )
+    (property "Footprint" "Pin_Headers:Pin_Header_Angled_1x02_Pitch2.54mm" (id 2) (at 99.06 109.22 0)
+      (effects (font (size 1.27 1.27)) hide)
+    )
+    (property "Datasheet" "~" (id 3) (at 99.06 109.22 0)
+      (effects (font (size 1.27 1.27)) hide)
+    )
+    (pin "1")
+    (pin "2")
+  )
+  (symbol (lib_id "HongFa:HFD2_005-S-L2-D") (at 138.43 80.01 0) (unit 1)
+    (in_bom yes) (on_board yes) (fields_autoplaced)
+    (property "Reference" "K1" (id 0) (at 154.94 73.5543 0))
+    (property "Value" "HFD2_005-S-L2-D" (id 1) (at 154.94 76.3294 0))
     (property "Footprint" "HFD2005SL2D" (id 2) (at 167.64 77.47 0)
       (effects (font (size 1.27 1.27)) (justify left) hide)
@@
     (pin "9")
   )
-  (symbol (lib_id "power:GND") (at 138.43 85.09 270) (unit 1)
-    (in_bom yes) (on_board yes)
-    (property "Reference" "#PWR0102" (id 0) (at 132.08 85.09 0)
-      (effects (font (size 1.27 1.27)) hide)
-    )
-    (property "Value" "GND" (id 1) (at 135.1788 85.217 90)
-      (effects (font (size 1.27 1.27)) (justify right))
-    )
-    (property "Footprint" "" (id 2) (at 138.43 85.09 0)
-      (effects (font (size 1.27 1.27)) hide)
-    )
-    (property "Datasheet" "" (id 3) (at 138.43 85.09 0)
-      (effects (font (size 1.27 1.27)) hide)
-    )
-    (pin "1")
-  )
-  (symbol (lib_id "Connector:Conn_01x02_Male") (at 181.61 82.55 180) (unit 1)
-    (in_bom yes) (on_board yes)
-    (property "Reference" "J1" (id 0) (at 182.3212 80.7212 0)
-      (effects (font (size 1.27 1.27)) (justify right))
-    )
-    (property "Value" "Conn_01x02_Male" (id 1) (at 178.8668 84.836 0)
-      (effects (font (size 1.27 1.27)) hide)
-    )
-    (property "Footprint" "Pin_Headers:Pin_Header_Angled_1x02_Pitch2.54mm" (id 2) (at 181.61 82.55 0)
-      (effects (font (size 1.27 1.27)) hide)
-    )
-    (property "Datasheet" "~" (id 3) (at 181.61 82.55 0)
-      (effects (font (size 1.27 1.27)) hide)
-    )
-    (pin "1")
-    (pin "2")
-  )
-  (symbol (lib_id "Connector:Conn_01x02_Male") (at 99.06 97.79 0) (unit 1)
-    (in_bom yes) (on_board yes)
-    (property "Reference" "J2" (id 0) (at 101.8032 93.1926 0))
-    (property "Value" "Power" (id 1) (at 101.6 102.87 0))
-    (property "Footprint" "Pin_Headers:Pin_Header_Angled_1x02_Pitch2.54mm" (id 2) (at 99.06 97.79 0)
-      (effects (font (size 1.27 1.27)) hide)
-    )
-    (property "Datasheet" "~" (id 3) (at 99.06 97.79 0)
-      (effects (font (size 1.27 1.27)) hide)
-    )
-    (pin "1")
-    (pin "2")
-  )
-  (symbol (lib_id "power:+5V") (at 121.92 97.79 0) (unit 1)
-    (in_bom yes) (on_board yes)
-    (property "Reference" "#PWR0103" (id 0) (at 121.92 101.6 0)
-      (effects (font (size 1.27 1.27)) hide)
-    )
-    (property "Value" "+5V" (id 1) (at 122.301 93.3958 0))
-    (property "Footprint" "" (id 2) (at 121.92 97.79 0)
-      (effects (font (size 1.27 1.27)) hide)
-    )
-    (property "Datasheet" "" (id 3) (at 121.92 97.79 0)
-      (effects (font (size 1.27 1.27)) hide)
-    )
-    (pin "1")
-  )
-  (symbol (lib_id "power:GND") (at 121.92 100.33 0) (unit 1)
-    (in_bom yes) (on_board yes)
-    (property "Reference" "#PWR0104" (id 0) (at 121.92 106.68 0)
-      (effects (font (size 1.27 1.27)) hide)
-    )
-    (property "Value" "GND" (id 1) (at 122.047 104.7242 0))
-    (property "Footprint" "" (id 2) (at 121.92 100.33 0)
-      (effects (font (size 1.27 1.27)) hide)
-    )
-    (property "Datasheet" "" (id 3) (at 121.92 100.33 0)
-      (effects (font (size 1.27 1.27)) hide)
-    )
-    (pin "1")
-  )
   (symbol (lib_id "power:+5V") (at 138.43 80.01 0) (unit 1)
-    (in_bom yes) (on_board yes)
+    (in_bom yes) (on_board yes) (fields_autoplaced)
     (property "Reference" "#PWR0105" (id 0) (at 138.43 83.82 0)
       (effects (font (size 1.27 1.27)) hide)
     )
-    (property "Value" "+5V" (id 1) (at 138.811 75.6158 0))
+    (property "Value" "+5V" (id 1) (at 138.43 76.4055 0))
     (property "Footprint" "" (id 2) (at 138.43 80.01 0)
       (effects (font (size 1.27 1.27)) hide)
@@
     )
     (pin "1")
-  )
-  (symbol (lib_id "Connector:Conn_01x02_Male") (at 99.06 109.22 0) (unit 1)
-    (in_bom yes) (on_board yes)
-    (property "Reference" "J3" (id 0) (at 101.8032 106.9594 0))
-    (property "Value" "Conn_01x02_Male" (id 1) (at 101.8032 106.934 0)
-      (effects (font (size 1.27 1.27)) hide)
-    )
-    (property "Footprint" "Pin_Headers:Pin_Header_Angled_1x02_Pitch2.54mm" (id 2) (at 99.06 109.22 0)
-      (effects (font (size 1.27 1.27)) hide)
-    )
-    (property "Datasheet" "~" (id 3) (at 99.06 109.22 0)
-      (effects (font (size 1.27 1.27)) hide)
-    )
-    (pin "1")
-    (pin "2")
   )
   (sheet_instances
@@
       (reference "#PWR0104") (unit 1) (value "GND") (footprint "")
     )
-    (path "/00000000-0000-0000-0000-000061269bbb"
+    (path "/e3d722df-9b54-4325-80d1-80f08f2b94b6"
       (reference "#PWR0105") (unit 1) (value "+5V") (footprint "")
     )
@@
       (reference "J3") (unit 1) (value "Conn_01x02_Male") (footprint "Pin_Headers:Pin_Header_Angled_1x02_Pitch2.54mm")
     )
-    (path "/00000000-0000-0000-0000-00006125b40d"
+    (path "/b82ab54a-4e5c-48e7-8792-ea0efee4329c"
       (reference "K1") (unit 1) (value "HFD2_005-S-L2-D") (footprint "HFD2005SL2D")
     )
